File: scr23-sens-to-can.kicad_sch (KiCad schematic)
At the start: 69 parts, among them J1 ATM13-12PA-BM01, U2 LM358_DFN, U3 LM358_DFN, U4 TJA1042T-3, U5 AP7370-33Y-13, U6 LM358_DFN, U7 LM358_DFN, U8 STM32G431CBT6, Y1 Crystal 4-48MHz, Y2 Crystal 32.768kHz

Commit message: add footprints
Parts:
- C1, C10, C11, C16, C17, C18, C19, C2, C20, C21, C22, C23, C3, C4, C5, C6, C7, C8, C9: footprint (none) -> Capacitor_SMD:C_0805_2012Metric
- C24, C25: renamed from C?; footprint (none) -> Capacitor_SMD:C_0805_2012Metric
- C28: renamed from C?; footprint TCJA_AVX -> (none)
- D1: renamed from D?; footprint (none) -> LED_SMD:LED_0402_1005Metric
- D11: footprint (none) -> LED_SMD:LED_0402_1005Metric
- R1, R10, R11, R12, R13, R14, R16, R17, R18, R2, R3, R4, R5, R6, R7, R8, R9: footprint (none) -> Resistor_SMD:R_0402_1005Metric
- R15: renamed from R?; footprint (none) -> Resistor_SMD:R_0402_1005Metric
- U5: footprint SOT89_B8D_DIO -> scr23-sens-to-can-main:AP7370-33Y-13
- U8: footprint LQFP48-7x7mm -> (none)
- gave numbers to parts that had none: 8
